File: modules/icesugar-nano-carrier/icesugar-nano-carrier.kicad_pcb (KiCad board)
At the start: 2 copper layers, 3 parts, among them J1 Conn_01x06_Pin, J2 Conn_01x06_Pin, J3 Conn_02x06_Odd_Even

Commit message: finish ICESugar Nano carrier board design
Parts:
- added M1: ~, MegaCastle:MegaCastle2x18-Module-I24.0x40.9-M800067FFF, F.Cu at (0.00, 3.41)
Connections:
- J1 pad 1: unconnected-(J1-Pin_1-Pad1) -> +3.3V
- J1 pad 2: unconnected-(J1-Pin_2-Pad2) -> GND
- J1 pad 3: unconnected-(J1-Pin_3-Pad3) -> A1
- J1 pad 4: unconnected-(J1-Pin_4-Pad4) -> B1
- J1 pad 5: unconnected-(J1-Pin_5-Pad5) -> D1
- J1 pad 6: unconnected-(J1-Pin_6-Pad6) -> E2
- J2 pad 1: unconnected-(J2-Pin_1-Pad1) -> B3
- J2 pad 2: unconnected-(J2-Pin_2-Pad2) -> A3
- J2 pad 3: unconnected-(J2-Pin_3-Pad3) -> B6
- J2 pad 4: unconnected-(J2-Pin_4-Pad4) -> C5
- J2 pad 5: unconnected-(J2-Pin_5-Pad5) -> GND
- J2 pad 6: unconnected-(J2-Pin_6-Pad6) -> +3.3V
- J3 pad 1: unconnected-(J3-Pin_1-Pad1) -> B4
- J3 pad 10: unconnected-(J3-Pin_10-Pad10) -> GND
- J3 pad 11: unconnected-(J3-Pin_11-Pad11) -> +3.3V
- J3 pad 12: unconnected-(J3-Pin_12-Pad12) -> +3.3V
- J3 pad 2: unconnected-(J3-Pin_2-Pad2) -> C6
- J3 pad 3: unconnected-(J3-Pin_3-Pad3) -> B5
- J3 pad 4: unconnected-(J3-Pin_4-Pad4) -> E3
- J3 pad 5: unconnected-(J3-Pin_5-Pad5) -> E1
- J3 pad 6: unconnected-(J3-Pin_6-Pad6) -> C2
- J3 pad 7: unconnected-(J3-Pin_7-Pad7) -> B1_DUP
- J3 pad 8: unconnected-(J3-Pin_8-Pad8) -> A1_DUP
- J3 pad 9: unconnected-(J3-Pin_9-Pad9) -> GND
Routing:
- net A1: track 0.00 -> 33.2 mm
- net E2: track 0.00 -> 28.9 mm
- net D1: track 0.00 -> 27.7 mm
- net B1: track 0.00 -> 27.2 mm
- net B1_DUP: track 0.00 -> 20.8 mm
- net E1: track 0.00 -> 15.9 mm
- net A1_DUP: track 0.00 -> 14.3 mm
- net C2: track 0.00 -> 11.4 mm
- net A3: track 0.00 -> 11.0 mm
- net C5: track 0.00 -> 10.7 mm
- net B6: track 0.00 -> 10.7 mm
- net B5: track 0.00 -> 10.6 mm
- net B3: track 0.00 -> 10.5 mm
- net E3: track 0.00 -> 9.61 mm
- net C6: track 0.00 -> 7.69 mm
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- added copper zone on F.Cu, net +3.3V
- added copper zone on B.Cu, net GND
Other:
- board outline added: 24 x 45.7 mm
- board text added: "3.3V"
- board text added: "A1"
- board text added: "A1'"
- board text added: "A3"
- board text added: "B1"
- board text added: "B1'"
- board text added: "B3"
- board text added: "B4"
- board text added: "B5"
- board text added: "B6"
- board text added: "C2"
- board text added: "C5"
- board text added: "C6"
- board text added: "D1"
- board text added: "E1"
- board text added: "E2"
- board text added: "E3"
- board text added: "GND"
- board text added: "MEGAphone iCESugar Nano Carrier 20250806 REMOVE U6, bridge with diode to power from 3.3V If not, 3.3V is OUTPUT not INPUT!!!"
